File: 01-power/kicad/ardustack-power.kicad_sch (KiCad schematic)
At the start: 14 parts, among them IC1 MC7805CTG, IC2 LP2950-33LPRE3, J1 CON-SOCJ-2155, P1 Power, P2 Analog, P3 Digital, P4 Digital, P5 CONN_01X01, P6 CONN_01X01, P7 CONN_01X01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

Commit message: Updates power, processor, and I/O boards to v1.0.0
Connections:
- net Vin: now also C1.1, IC1.1 (INPUT), J1.1
Changed lines of the file:
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@@
   (junction (at 139.7 101.6) (diameter 0) (color 0 0 0 0)
+  )
+  (junction (at 76.2 101.6) (diameter 0) (color 0 0 0 0)
   )
   (junction (at 236.22 55.88) (diameter 1.016) (color 0 0 0 0)
@@
     (stroke (width 0) (type solid) (color 0 0 0 0))
   )
+  (wire (pts (xy 76.2 99.06) (xy 76.2 101.6))
+    (stroke (width 0) (type default) (color 0 0 0 0))
+  )
   (wire (pts (xy 119.38 101.6) (xy 139.7 101.6))
     (stroke (width 0) (type default) (color 0 0 0 0))
@@
   (wire (pts (xy 238.76 53.34) (xy 236.22 53.34))
     (stroke (width 0) (type solid) (color 0 0 0 0))
+  )
+  (wire (pts (xy 76.2 101.6) (xy 88.9 101.6))
+    (stroke (width 0) (type default) (color 0 0 0 0))
   )
   (wire (pts (xy 259.08 53.34) (xy 267.97 53.34))
@@
     (stroke (width 0) (type solid) (color 0 0 0 0))
   )
-  (wire (pts (xy 63.5 101.6) (xy 88.9 101.6))
+  (wire (pts (xy 63.5 101.6) (xy 76.2 101.6))
     (stroke (width 0) (type default) (color 0 0 0 0))
   )
@@
     (effects (font (size 1.524 1.524)) (justify left bottom))
   )
+  (label "Vin" (at 76.2 99.06 0)
+    (effects (font (size 1.27 1.27)) (justify left bottom))
+  )
   (label "4" (at 267.97 66.04 0)
