File: 02-processor/kicad/ardustack-mcu.kicad_sch (KiCad schematic)
At the start: 15 parts, among them J1 1-2199298-9, P1 Power, P2 Analog, P3 Digital, P4 Digital, P5 CONN_01X01, P6 CONN_01X01, P7 CONN_01X01, P8 CONN_01X01, Y1 ABL-16.000MHZ-B2

Commit message: Updates power, processor, and I/O boards to v1.0.0
Connections:
- net IOREF is gone; now on net +5V: P1.2 (Pin_2)
Changed lines of the file:
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@@
     (stroke (width 0) (type solid) (color 0 0 0 0))
+  )
+  (wire (pts (xy 121.92 71.12) (xy 124.46 71.12))
+    (stroke (width 0) (type default) (color 0 0 0 0))
   )
   (wire (pts (xy 229.87 50.8) (xy 229.87 34.29))
@@
     (effects (font (size 1.27 1.27)) (justify left bottom))
   )
+  (label "IOREF" (at 121.92 71.12 180)
+    (effects (font (size 1.27 1.27)) (justify right bottom))
+  )
   (label "8" (at 267.97 53.34 0)
