File: 03-input-output/kicad/ardustack-io.kicad_pcb (KiCad board)
At the start: 2 copper layers, 68.6 x 53.3 mm, 14 parts, among them J1 825437-6, P1 Power, P2 Analog, P3 Digital, P4 Digital, P5 CONN_01X01, P6 CONN_01X01, P7 CONN_01X01, P8 CONN_01X01

Commit message: Updates Ardustack I/O board PCB silkscreen
Parts:
- added G***: LOGO, ardustack-io:emblem, B.Cu at (167.0, 102.0)
- added G***: LOGO, ardustack-io:name_plate, B.Cu at (144.0, 102.0)

Commit message: Updates PCBs with name and version
Other:
- board text added: "ARDUSTACK I/O PCB v0.9.0"
Changed lines of the file:
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@@
   (gr_line (start 175.514 73.025) (end 110.998 73.025) (layer "Edge.Cuts") (width 0.15))
   (gr_line (start 177.038 85.979) (end 177.038 74.549) (layer "Edge.Cuts") (width 0.15))
+  (gr_text "ARDUSTACK I/O PCB v0.9.0" (at 144.3 110.1) (layer "B.SilkS")
+    (effects (font (size 1 1) (thickness 0.15)) (justify mirror))
+  )
   (gr_text "Reset" (at 144.018 120 90) (layer "F.SilkS")
     (effects (font (size 1 1) (thickness 0.15)))

Commit message: Updates power, processor, and I/O boards to v1.0.0
Connections:
- J1 pad 3: +5V -> /Vin
Routing:
- net /Vin: track 0.00 -> 47.2 mm
- net +5V: track 42.4 -> 27.7 mm
Other:
- board text added: "(+3V3)"
- board text added: "(2)"
- board text added: "(3)"
- board text added: "(4)"
- board text added: "(5)"
- board text added: "(6)"
- board text added: "(7)"
- board text added: "(8)"
- board text added: "(9)"
- board text added: "(A0)"
- board text added: "(A1)"
- board text added: "(A2)"
- board text added: "(A3)"
- board text added: "(AREF)"
- board text added: "(IOREF)"
- board text added: "(MISO)"
- board text added: "(MOSI)"
- board text added: "(SCL)"
- board text added: "(SDA)"
- board text added: "(SS)"
- board text added: "ARDUSTACK I/O PCB v1.0.0"
- board text added: "GND"
- board text added: "NC"
- board text added: "Vin"
- board text removed: "ARDUSTACK I/O PCB v0.9.0"
Changed lines of the file:
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@@
     (property "Sheetname" "")
     (attr through_hole)
-    (fp_text reference "R2" (at 0 -2.5) (layer "F.SilkS")
+    (fp_text reference "R2" (at -2.52 2.286) (layer "F.SilkS")
       (effects (font (size 1.27 1.27) (thickness 0.254)))
     )
@@
       (effects (font (size 1.27 1.27) (thickness 0.254)))
     )
-    (fp_text user "${REFERENCE}" (at 0 -2.5) (layer "F.Fab")
+    (fp_text user "${REFERENCE}" (at -2.52 2.286) (layer "F.Fab")
       (effects (font (size 1.27 1.27) (thickness 0.254)))
     )
@@
     (property "Sheetname" "")
     (attr through_hole)
-    (fp_text reference "C1" (at 0 3.5) (layer "F.SilkS")
+    (fp_text reference "C1" (at -4.6 0) (layer "F.SilkS")
       (effects (font (size 1.27 1.27) (thickness 0.254)))
     )
@@
       (effects (font (size 1.27 1.27) (thickness 0.254)))
     )
-    (fp_text user "${REFERENCE}" (at 0 3.5) (layer "F.Fab")
+    (fp_text user "${REFERENCE}" (at -4.6 0) (layer "F.Fab")
       (effects (font (size 1.27 1.27) (thickness 0.254)))
     )
@@
     (property "Sheetname" "")
     (attr through_hole)
-    (fp_text reference "S1" (at 0 5) (layer "F.SilkS")
+    (fp_text reference "S1" (at 0 4.6) (layer "F.SilkS")
       (effects (font (size 1.27 1.27) (thickness 0.254)))
     )
@@
       (effects (font (size 1.27 1.27) (thickness 0.254)))
     )
-    (fp_text user "${REFERENCE}" (at 0 5) (layer "F.Fab")
+    (fp_text user "${REFERENCE}" (at 0 4.6) (layer "F.Fab")
       (effects (font (size 1.27 1.27) (thickness 0.254)))
     )
@@
     (property "Sheetname" "")
     (attr through_hole)
-    (fp_text reference "J1" (at 0 3 90) (layer "F.SilkS")
+    (fp_text reference "J1" (at 0 2.8 90) (layer "F.SilkS")
       (effects (font (size 1.27 1.27) (thickness 0.254)))
     )
@@
       (effects (font (size 1.27 1.27) (thickness 0.254)))
     )
-    (fp_text user "${REFERENCE}" (at 0 3 90) (layer "F.Fab")
+    (fp_text user "${REFERENCE}" (at 0 2.8 90) (layer "F.Fab")
       (effects (font (size 1.27 1.27) (thickness 0.254)))
     )
@@
       (net 4 "GND") (pinfunction "2") (pintype "passive"))
     (pad "3" thru_hole circle (at -1.27 0 90) (size 1.59 1.59) (drill 1.09) (layers *.Cu *.Mask)
-      (net 3 "+5V") (pinfunction "3") (pintype "passive"))
+      (net 5 "/Vin") (pinfunction "3") (pintype "passive"))
     (pad "4" thru_hole circle (at 1.27 0 90) (size 1.59 1.59) (drill 1.09) (layers *.Cu *.Mask)
       (net 22 "/0(Rx)") (pinfunction "4") (pintype "passive"))
@@
   (gr_line (start 175.514 73.025) (end 110.998 73.025) (layer "Edge.Cuts") (width 0.15))
   (gr_line (start 177.038 85.979) (end 177.038 74.549) (layer "Edge.Cuts") (width 0.15))
-  (gr_text "ARDUSTACK I/O PCB v0.9.0" (at 144.3 110.1) (layer "B.SilkS")
+  (gr_text "ARDUSTACK I/O PCB v1.0.0" (at 144.3 110.1) (layer "B.SilkS")
     (effects (font (size 1 1) (thickness 0.15)) (justify mirror))
   )
-  (gr_text "Reset" (at 144.018 120 90) (layer "F.SilkS")
+  (gr_text "(A2)" (at 166.878 119.5 90) (layer "F.SilkS")
     (effects (font (size 1 1) (thickness 0.15)))
   )
-  (gr_text "+5V" (at 149.098 120 90) (layer "F.SilkS")
+  (gr_text "NC" (at 132.334 79.6 90) (layer "F.SilkS")
     (effects (font (size 1 1) (thickness 0.15)))
   )
-  (gr_text "Rx" (at 174.498 79.2 90) (layer "F.SilkS")
+  (gr_text "(AREF)" (at 134.874 79.6 90) (layer "F.SilkS")
     (effects (font (size 1 1) (thickness 0.15)))
   )
-  (gr_text "13" (at 139.954 79.2 90) (layer "F.SilkS")
+  (gr_text "(SS)" (at 147.574 79.6 90) (layer "F.SilkS")
     (effects (font (size 1 1) (thickness 0.15)))
   )
-  (gr_text "Tx" (at 171.958 79.2 90) (layer "F.SilkS")
+  (gr_text "Vin" (at 156.718 119.5 90) (layer "F.SilkS")
+    (effects (font (size 1 1) (thickness 0.15)))
+  )
+  (gr_text "(5)" (at 161.798 79.6 90) (layer "F.SilkS")
+    (effects (font (size 1 1) (thickness 0.15)))
+  )
+  (gr_text "NC" (at 138.938 119.5 90) (layer "F.SilkS")
+    (effects (font (size 1 1) (thickness 0.15)))
+  )
+  (gr_text "Reset" (at 144.018 119.5 90) (layer "F.SilkS")
+    (effects (font (size 1 1) (thickness 0.15)))
+  )
+  (gr_text "(6)" (at 159.258 79.6 90) (layer "F.SilkS")
+    (effects (font (size 1 1) (thickness 0.15)))
+  )
+  (gr_text "(SCL)" (at 174.098 119.5 90) (layer "F.SilkS")
+    (effects (font (size 1 1) (thickness 0.15)))
+  )
+  (gr_text "(3)" (at 166.878 79.6 90) (layer "F.SilkS")
+    (effects (font (size 1 1) (thickness 0.15)))
+  )
+  (gr_text "(7)" (at 156.718 79.6 90) (layer "F.SilkS")
+    (effects (font (size 1 1) (thickness 0.15)))
+  )
+  (gr_text "(A1)" (at 164.338 119.5 90) (layer "F.SilkS")
+    (effects (font (size 1 1) (thickness 0.15)))
+  )
+  (gr_text "(MOSI)" (at 145.034 79.6 90) (layer "F.SilkS")
+    (effects (font (size 1 1) (thickness 0.15)))
+  )
+  (gr_text "GND" (at 137.414 79.6 90) (layer "F.SilkS")
+    (effects (font (size 1 1) (thickness 0.15)))
+  )
+  (gr_text "(SDA)" (at 171.958 119.5 90) (layer "F.SilkS")
+    (effects (font (size 1 1) (thickness 0.15)))
+  )
+  (gr_text "(4)" (at 164.338 79.6 90) (layer "F.SilkS")
+    (effects (font (size 1 1) (thickness 0.15)))
+  )
+  (gr_text "(2)" (at 169.418 79.6 90) (layer "F.SilkS")
+    (effects (font (size 1 1) (thickness 0.15)))
+  )
+  (gr_text "(A3)" (at 169.418 119.5 90) (layer "F.SilkS")
+    (effects (font (size 1 1) (thickness 0.15)))
+  )
+  (gr_text "(+3V3)" (at 146.558 119.5 90) (layer "F.SilkS")
+    (effects (font (size 1 1) (thickness 0.15)))
+  )
+  (gr_text "+5V" (at 149.098 119.5 90) (layer "F.SilkS")
+    (effects (font (size 1 1) (thickness 0.15)))
+  )
+  (gr_text "(8)" (at 152.654 79.6 90) (layer "F.SilkS")
+    (effects (font (size 1 1) (thickness 0.15)))
+  )
+  (gr_text "(MISO)" (at 142.494 79.6 90) (layer "F.SilkS")
+    (effects (font (size 1 1) (thickness 0.15)))
+  )
+  (gr_text "(A0)" (at 161.798 119.5 90) (layer "F.SilkS")
+    (effects (font (size 1 1) (thickness 0.15)))
+  )
+  (gr_text "Rx" (at 174.498 79.6 90) (layer "F.SilkS")
+    (effects (font (size 1 1) (thickness 0.15)))
+  )
+  (gr_text "(IOREF)" (at 141.478 119.5 90) (layer "F.SilkS")
+    (effects (font (size 1 1) (thickness 0.15)))
+  )
+  (gr_text "13" (at 139.954 79.6 90) (layer "F.SilkS")
+    (effects (font (size 1 1) (thickness 0.15)))
+  )
+  (gr_text "GND" (at 154.178 119.5 90) (layer "F.SilkS")
+    (effects (font (size 1 1) (thickness 0.15)))
+  )
+  (gr_text "NC" (at 129.794 79.6 90) (layer "F.SilkS")
+    (effects (font (size 1 1) (thickness 0.15)))
+  )
+  (gr_text "GND" (at 151.638 119.5 90) (layer "F.SilkS")
+    (effects (font (size 1 1) (thickness 0.15)))
+  )
+  (gr_text "(9)" (at 150.114 79.6 90) (layer "F.SilkS")
+    (effects (font (size 1 1) (thickness 0.15)))
+  )
+  (gr_text "Tx" (at 171.958 79.6 90) (layer "F.SilkS")
     (effects (font (size 1 1) (thickness 0.15)))
   )
@@
   (segment (start 144.018 123.825) (end 113.075489 92.882489) (width 0.25) (layer "F.Cu") (net 2))
   (segment (start 129.45 104.5) (end 148.775 123.825) (width 0.25) (layer "F.Cu") (net 3))
-  (segment (start 129.45 99.72) (end 129.45 104.5) (width 0.25) (layer "F.Cu") (net 3))
-  (segment (start 122.4 92.67) (end 129.45 99.72) (width 0.25) (layer "F.Cu") (net 3))
   (segment (start 148.775 123.825) (end 149.098 123.825) (width 0.25) (layer "F.Cu") (net 3))
+  (segment (start 125.563 92.67) (end 156.718 123.825) (width 0.25) (layer "F.Cu") (net 5))
+  (segment (start 122.4 92.67) (end 125.563 92.67) (width 0.25) (layer "F.Cu") (net 5))
   (segment (start 122.4 87.59) (end 124.334511 89.524511) (width 0.25) (layer "F.Cu") (net 21))
   (segment (start 124.334511 89.524511) (end 157.998489 89.524511) (width 0.25) (layer "F.Cu") (net 21))
