File: 03-input-output/kicad/ardustack-io.kicad_sch (KiCad schematic)
At the start: 14 parts, among them J1 825437-6, P1 Power, P2 Analog, P3 Digital, P4 Digital, P5 CONN_01X01, P6 CONN_01X01, P7 CONN_01X01, P8 CONN_01X01

Commit message: Updates power, processor, and I/O boards to v1.0.0
Connections:
- net +5V: no longer J1.3
- net Vin: now also J1.3
Changed lines of the file:
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@@
     (effects (font (size 1.524 1.524)) (justify left bottom))
+  )
+  (label "Vin" (at 101.6 119.38 180)
+    (effects (font (size 1.27 1.27)) (justify right bottom))
   )
   (label "A4(SDA)" (at 226.06 73.66 0)
@@
     (pin "6")
   )
-  (symbol (lib_id "power:+5V") (at 101.6 119.38 0) (unit 1)
-    (in_bom yes) (on_board yes) (fields_autoplaced)
-    (property "Reference" "#PWR05" (id 0) (at 101.6 123.19 0)
-      (effects (font (size 1.27 1.27)) hide)
-    )
-    (property "Value" "+5V" (id 1) (at 101.6 114.3 0))
-    (property "Footprint" "" (id 2) (at 101.6 119.38 0)
-      (effects (font (size 1.27 1.27)) hide)
-    )
-    (property "Datasheet" "" (id 3) (at 101.6 119.38 0)
-      (effects (font (size 1.27 1.27)) hide)
-    )
-    (pin "1")
-  )
   (symbol (lib_id "ardustack-io:CFR-25JR-52-10K") (at 111.76 66.04 270) (unit 1)
     (in_bom yes) (on_board yes) (fields_autoplaced)
@@
       (reference "#PWR04") (unit 1) (value "GND") (footprint "")
     )
-    (path "/7ee42005-9b48-4c21-8e5a-15d6306c2fc3"
-      (reference "#PWR05") (unit 1) (value "+5V") (footprint "")
-    )
     (path "/efa43d59-2d48-4937-9902-b541a7d28faa"
